File: breadboard_clock.sch (KiCad schematic (older format))
At the start: 26 parts, among them SW101 SW_Push, SW102 SW_SPDT, U101 ICM7555, U102 74LS04, U103 74LS04, U104 74LS08, U105 74LS32, U106 ICM7555, U107 74LS04, U108 ICM7555

Commit message: Add files via upload
Parts:
- added J101: Conn_01x02_Male, Connector_PinHeader_2.54mm:PinHeader_1x02_P2.54mm_Vertical_SMD_Pin1Right, symbol Connector:Conn_01x02_Male
- SW101: footprint (none) -> Button_Switch_SMD:SW_SPST_B3S-1000
- SW102: footprint (none) -> Button_Switch_SMD:SW_SPDT_PCM12
- e101: renamed from e; footprint (none) -> Gerig-Added:Potentiomter_Bourns_PDB12_THT
Connections:
- net GND: now also J101.2 (Pin_2)
- net VCC: now also J101.1 (Pin_1)
Other:
- note added: "0"
- note added: "1"
- note added: "29 Jan 2021"
- note added: "Based off Ben Eater's Breadboard clock module: eater.net/8bit/clock"
- note added: "Breadboard Clock Module"
Changed lines of the file:
@@
 $EndComp
 $Comp
-L Device:R_POT e
+L Device:R_POT e101
 U 1 1 6015012D
 P 3450 1650
-F 0 "e" H 3380 1604 50  0000 R CNN
+F 0 "e101" H 3380 1604 50  0000 R CNN
 F 1 "R_POT" H 3380 1695 50  0000 R CNN
-F 2 "" H 3450 1650 50  0001 C CNN
+F 2 "Gerig-Added:Potentiomter_Bourns_PDB12_THT" H 3450 1650 50  0001 C CNN
 F 3 "~" H 3450 1650 50  0001 C CNN
 	1    3450 1650
@@
 F 0 "SW101" H 4600 1785 50  0000 C CNN
 F 1 "SW_Push" H 4600 1694 50  0000 C CNN
-F 2 "" H 4600 1700 50  0001 C CNN
+F 2 "Button_Switch_SMD:SW_SPST_B3S-1000" H 4600 1700 50  0001 C CNN
 F 3 "~" H 4600 1700 50  0001 C CNN
 	1    4600 1500
@@
 F 0 "SW102" H 7800 2085 50  0000 C CNN
 F 1 "SW_SPDT" H 7800 1994 50  0000 C CNN
-F 2 "" H 7800 1800 50  0001 C CNN
+F 2 "Button_Switch_SMD:SW_SPDT_PCM12" H 7800 1800 50  0001 C CNN
 F 3 "~" H 7800 1800 50  0001 C CNN
 	1    7800 1800
@@
 Wire Wire Line
 	8050 3800 8500 3800
+Text Notes 7350 7500 0    50   ~ 0
+Breadboard Clock Module
+Text Notes 8150 7650 0    50   ~ 0
+29 Jan 2021
+Text Notes 7050 6650 0    50   ~ 0
+Based off Ben Eater's Breadboard clock module: eater.net/8bit/clock
+Text Notes 7280 7250 0    50   ~ 0
+1
+Text Notes 7380 7250 0    50   ~ 0
+1
+Text Notes 10550 7650 0    50   ~ 0
+0
+$Comp
+L power:VCC #PWR0110
+U 1 1 6040569A
+P 9800 3900
+F 0 "#PWR0110" H 9800 3750 50  0001 C CNN
+F 1 "VCC" H 9700 4000 50  0000 C CNN
+F 2 "Connector_PinHeader_2.54mm:PinHeader_1x02_P2.54mm_Vertical" H 9800 3900 50  0001 C CNN
+F 3 "" H 9800 3900 50  0001 C CNN
+	1    9800 3900
+	1    0    0    -1
+$EndComp
+$Comp
+L power:GND #PWR0111
+U 1 1 60406039
+P 9900 3900
+F 0 "#PWR0111" H 9900 3650 50  0001 C CNN
+F 1 "GND" H 9750 3800 50  0000 C CNN
+F 2 "Connector_PinHeader_2.54mm:PinHeader_1x02_P2.54mm_Vertical" H 9900 3900 50  0001 C CNN
+F 3 "" H 9900 3900 50  0001 C CNN
+	1    9900 3900
+	-1   0    0    1
+$EndComp
+$Comp
+L Connector:Conn_01x02_Male J101
+U 1 1 6040D82B
+P 9800 4100
+F 0 "J101" V 9954 3912 50  0000 R CNN
+F 1 "Conn_01x02_Male" V 9863 3912 50  0000 R CNN
+F 2 "Connector_PinHeader_2.54mm:PinHeader_1x02_P2.54mm_Vertical_SMD_Pin1Right" V 9817 3912 50  0001 R CNN
+F 3 "~" H 9800 4100 50  0001 C CNN
+	1    9800 4100
+	0    -1   -1   0
+$EndComp
 $EndSCHEMATC

Commit message: Add files via upload
Parts:
- added D1, D2, D4: LED, LED_SMD:LED_0805_2012Metric, symbol Device:LED
- added J2: Conn_01x03_Male, Connector_PinHeader_2.54mm:PinHeader_1x03_P2.54mm_Vertical_SMD_Pin1Right, symbol Connector:Conn_01x03_Male
- added R10, R3, R6: 220, Resistor_SMD:R_0805_2012Metric, symbol Device:R
- renumbered C101 to C1, C102 to C2, C103 to C3, C104 to C4, C105 to C5, C106 to C6, C107 to C7, D101 to D3, J101 to J1, e101 to P1, R101 to R1, R102 to R2, R103 to R4, R104 to R5, R105 to R7, R106 to R8, R107 to R9, SW101 to SW1, SW102 to SW2, U101 to U1, U102 to U2, U103 to U3, U104 to U4, U106 to U5, U105 to U6, U107 to U7, U108 to U8
Connections:
- net CLK: now also J2.1 (Pin_1)
- net GND: now also J2.3 (Pin_3), R10.2, R3.2, R6.2
- net ~CLK: now also J2.2 (Pin_2)
- net at U1.3 (Q), U4.1: now also D1.2 (A)
- net at U4.5, U5.3 (Q): now also D2.2 (A)
- net at U3.1, U4.2, U8.3 (Q): now also D4.2 (A)
- new net: D1.1 (K), R3.1
- new net: D2.1 (K), R6.1
- new net: D4.1 (K), R10.1
Other:
- note added: "Clock/ ~Clock output"
- note added: "Power/GND input"
- moved on the sheet: C1, C2, C3, C4, P1, R1, R2, R4, R5, SW1, U1, U5
